Commit message: added darker shades of color to differentiate in bot view (can be run with test_world_4_robots_colorful.launch file)

File: models/turtlebot3_blue.gazebo.xacro (robot description, xacro)
@@ -93,5 +93,5 @@
   </gazebo>
   <gazebo reference="base_scan">
-    <material>Gazebo/Blue</material>
+    <material>Gazebo/FlatBlack</material>
     <sensor type="ray" name="lds_lfcd_sensor">
       <pose>0 0 0 0 0 0</pose>

File: models/turtlebot3_darkblue.gazebo.xacro (robot description, xacro)
@@ -4,5 +4,10 @@
   <xacro:arg name="imu_visual"   default="false"/>
   <gazebo reference="base_link">
-    <material>Gazebo/Red</material>
+    <visual>
+      <material>
+        <ambient>0 0 0.75 1</ambient>   <!-- Dark blue with full opacity -->
+        <diffuse>0 0 0.75 1</diffuse>   <!-- Dark blue with full opacity -->
+      </material>
+    </visual>
   </gazebo>
   <gazebo reference="wheel_left_link">

File: models/turtlebot3_darkred.gazebo.xacro (robot description, xacro)
@@ -3,7 +3,12 @@
   <xacro:arg name="laser_visual" default="false"/>
   <xacro:arg name="imu_visual"   default="false"/>
-  <gazebo reference="base_link">
-    <material>Gazebo/Red</material>
-  </gazebo>
+<gazebo reference="base_link">
+  <visual>
+    <material>
+      <ambient>0.75 0 0 1</ambient>   <!-- Dark red with full opacity -->
+      <diffuse>0.75 0 0 1</diffuse>   <!-- Dark red with full opacity -->
+    </material>
+  </visual>
+</gazebo>
   <gazebo reference="wheel_left_link">
     <mu1>0.1</mu1>
