Commit message: change dark b/r to green/yellow

File: models/turtlebot3_darkred.urdf.xacro (robot description, xacro)
@@ -15,5 +15,5 @@
         <mesh filename="package://turtlebot3_description/meshes/bases/burger_base.stl" scale="0.001 0.001 0.001"/>
       </geometry>
-      <material name="red"/>
+      <material name="yellow"/>
     </visual>
     <collision>

File: models/turtlebot3_green.gazebo.xacro (robot description, xacro)
@@ -3,12 +3,7 @@
   <xacro:arg name="laser_visual" default="false"/>
   <xacro:arg name="imu_visual"   default="false"/>
-<gazebo reference="base_link">
-  <visual>
-    <material>
-      <ambient>0.7 0 0 1</ambient>   <!-- Dark red with full opacity -->
-      <diffuse>0.7 0 0 1</diffuse>   <!-- Dark red with full opacity -->
-    </material>
-  </visual>
-</gazebo>
+  <gazebo reference="base_link">
+    <material>Gazebo/Green</material>
+  </gazebo>
   <gazebo reference="wheel_left_link">
     <mu1>0.1</mu1>

File: models/turtlebot3_green.urdf.xacro (robot description, xacro)
@@ -15,5 +15,5 @@
         <mesh filename="package://turtlebot3_description/meshes/bases/burger_base.stl" scale="0.001 0.001 0.001"/>
       </geometry>
-      <material name="red"/>
+      <material name="green"/>
     </visual>
     <collision>

File: models/turtlebot3_yellow.gazebo.xacro (robot description, xacro)
@@ -3,12 +3,7 @@
   <xacro:arg name="laser_visual" default="false"/>
   <xacro:arg name="imu_visual"   default="false"/>
-  <gazebo reference="base_link">
-    <visual>
-      <material>
-        <ambient>0 0 0.7 1</ambient>   <!-- Dark blue with full opacity -->
-        <diffuse>0 0 0.7 1</diffuse>   <!-- Dark blue with full opacity -->
-      </material>
-    </visual>
-  </gazebo>
+<gazebo reference="base_link">
+  <material>Gazebo/Yellow</material>
+</gazebo>
   <gazebo reference="wheel_left_link">
     <mu1>0.1</mu1>
