Commit message: Added a lot of stuff

File: models/turtlebot3_darkblue.gazebo.xacro (robot description, xacro)
@@ -4,5 +4,10 @@
   <xacro:arg name="imu_visual"   default="false"/>
   <gazebo reference="base_link">
-    <material>Gazebo/Green</material>
+    <visual>
+      <material>
+        <ambient>0 0 0.75 1</ambient>   <!-- Dark blue with full opacity -->
+        <diffuse>0 0 0.75 1</diffuse>   <!-- Dark blue with full opacity -->
+      </material>
+    </visual>
   </gazebo>
   <gazebo reference="wheel_left_link">

File: models/turtlebot3_darkblue.urdf.xacro (robot description, xacro)
@@ -2,5 +2,5 @@
 <robot name="turtlebot3_model1" xmlns:xacro="http://ros.org/wiki/xacro">
   <xacro:include filename="$(find turtlebot3_description)/urdf/common_properties.xacro"/>
-  <xacro:include filename="$(find cs_bot)/models/turtlebot3_darkred.gazebo.xacro"/>
+  <xacro:include filename="$(find cs_bot)/models/turtlebot3_darkblue.gazebo.xacro"/>
   <link name="base_footprint"/>
   <joint name="base_joint" type="fixed">
@@ -15,5 +15,5 @@
         <mesh filename="package://turtlebot3_description/meshes/bases/burger_base.stl" scale="0.001 0.001 0.001"/>
       </geometry>
-      <material name="yellow"/>
+      <material name="red"/>
     </visual>
     <collision>

File: models/turtlebot3_darkred.gazebo.xacro (robot description, xacro)
@@ -4,5 +4,10 @@
   <xacro:arg name="imu_visual"   default="false"/>
 <gazebo reference="base_link">
-  <material>Gazebo/Yellow</material>
+  <visual>
+    <material>
+      <ambient>0.75 0 0 1</ambient>   <!-- Dark red with full opacity -->
+      <diffuse>0.75 0 0 1</diffuse>   <!-- Dark red with full opacity -->
+    </material>
+  </visual>
 </gazebo>
   <gazebo reference="wheel_left_link">

File: models/turtlebot3_darkred.urdf.xacro (robot description, xacro)
@@ -2,5 +2,5 @@
 <robot name="turtlebot3_model1" xmlns:xacro="http://ros.org/wiki/xacro">
   <xacro:include filename="$(find turtlebot3_description)/urdf/common_properties.xacro"/>
-  <xacro:include filename="$(find cs_bot)/models/turtlebot3_darkblue.gazebo.xacro"/>
+  <xacro:include filename="$(find cs_bot)/models/turtlebot3_darkred.gazebo.xacro"/>
   <link name="base_footprint"/>
   <joint name="base_joint" type="fixed">
@@ -15,5 +15,5 @@
         <mesh filename="package://turtlebot3_description/meshes/bases/burger_base.stl" scale="0.001 0.001 0.001"/>
       </geometry>
-      <material name="green"/>
+      <material name="red"/>
     </visual>
     <collision>
